File: SMD-Transistor-Blinker.kicad_sch (KiCad schematic)
At the start: 12 parts, among them J1 Conn_01x02_Pin, J4 PINHD_1x1_Male, Q1 BC846, Q2 BC846

Commit message: optimierung kicad
Other:
- moved on the sheet: J1, J4
Changed lines of the file:
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@@
-	)
-	(junction
-		(at 148.59 81.28)
-		(diameter 0)
-		(color 0 0 0 0)
 	)
 	(junction
@@
 	)
 	(junction
-		(at 148.59 124.46)
-		(diameter 0)
-		(color 0 0 0 0)
-	)
-	(junction
 		(at 203.2 81.28)
 		(diameter 0)
@@
 	)
 	(junction
+		(at 166.37 124.46)
+		(diameter 0)
+		(color 0 0 0 0)
+	)
+	(junction
 		(at 203.2 100.33)
+		(diameter 0)
+		(color 0 0 0 0)
+	)
+	(junction
+		(at 166.37 81.28)
 		(diameter 0)
 		(color 0 0 0 0)
@@
 	(wire
 		(pts
-			(xy 148.59 105.41) (xy 148.59 124.46)
+			(xy 166.37 105.41) (xy 166.37 124.46)
 		)
 		(stroke
@@
 	(wire
 		(pts
-			(xy 148.59 102.87) (xy 148.59 81.28)
+			(xy 166.37 102.87) (xy 166.37 81.28)
 		)
 		(stroke
@@
 	(wire
 		(pts
+			(xy 166.37 124.46) (xy 179.07 124.46)
+		)
+		(stroke
+			(width 0)
+			(type default)
+		)
+	)
+	(wire
+		(pts
 			(xy 186.69 113.03) (xy 190.5 113.03)
 		)
@@
 	(wire
 		(pts
-			(xy 129.54 105.41) (xy 148.59 105.41)
+			(xy 160.02 105.41) (xy 166.37 105.41)
 		)
 		(stroke
@@
 	(wire
 		(pts
-			(xy 248.92 124.46) (xy 217.17 124.46)
+			(xy 222.25 124.46) (xy 217.17 124.46)
 		)
 		(stroke
@@
 	(wire
 		(pts
-			(xy 148.59 124.46) (xy 179.07 124.46)
-		)
-		(stroke
-			(width 0)
-			(type default)
-		)
-	)
-	(wire
-		(pts
 			(xy 190.5 100.33) (xy 190.5 88.9)
 		)
@@
 	(wire
 		(pts
-			(xy 129.54 102.87) (xy 148.59 102.87)
-		)
-		(stroke
-			(width 0)
-			(type default)
-		)
-	)
-	(wire
-		(pts
-			(xy 148.59 81.28) (xy 179.07 81.28)
+			(xy 160.02 102.87) (xy 166.37 102.87)
 		)
 		(stroke
@@
 		)
 	)
-	(netclass_flag ""
-		(length 2.54)
-		(shape round)
-		(at 153.67 81.28 0)
-		(fields_autoplaced yes)
-		(effects
-			(font
-				(size 1.27 1.27)
-			)
-			(justify left bottom)
-		)
-		(property "Netclass" "supply"
-			(at 154.3685 78.74 0)
-			(effects
-				(font
-					(size 1.27 1.27)
-					(italic yes)
-				)
-				(justify left)
-			)
-		)
-	)
-	(netclass_flag ""
-		(length 2.54)
-		(shape round)
-		(at 156.21 124.46 180)
-		(effects
-			(font
-				(size 1.27 1.27)
-			)
-			(justify right bottom)
-		)
-		(property "Netclass" "supply"
-			(at 155.702 126.746 0)
-			(effects
-				(font
-					(size 1.27 1.27)
-					(italic yes)
-				)
-				(justify right)
-			)
+	(wire
+		(pts
+			(xy 166.37 81.28) (xy 179.07 81.28)
+		)
+		(stroke
+			(width 0)
+			(type default)
 		)
 	)
@@
 	)
 	(symbol
+		(lib_name "PWR_FLAG_1")
 		(lib_id "power:PWR_FLAG")
-		(at 148.59 124.46 180)
+		(at 166.37 124.46 180)
 		(unit 1)
 		(exclude_from_sim no)
@@
 		(fields_autoplaced yes)
 		(property "Reference" "#FLG02"
-			(at 148.59 126.365 0)
+			(at 166.37 126.365 0)
 			(effects
 				(font
@@
 		)
 		(property "Value" "PWR_FLAG"
-			(at 148.59 129.54 0)
+			(at 166.37 129.54 0)
 			(effects
 				(font
@@
 		)
 		(property "Footprint" ""
-			(at 148.59 124.46 0)
+			(at 166.37 124.46 0)
 			(effects
 				(font
@@
 		)
 		(property "Datasheet" "~"
-			(at 148.59 124.46 0)
-			(effects
-				(font
-					(size 1.27 1.27)
-				)
-				(hide yes)
-			)
-		)
-		(property "Description" ""
-			(at 148.59 124.46 0)
+			(at 166.37 124.46 0)
+			(effects
+				(font
+					(size 1.27 1.27)
+				)
+				(hide yes)
+			)
+		)
+		(property "Description" "Special symbol for telling ERC where power comes from"
+			(at 166.37 124.46 0)
 			(effects
 				(font
@@
 			)
 		)
+		(property "Sim.Device" "D"
+			(at 217.17 95.25 0)
+			(effects
+				(font
+					(size 1.27 1.27)
+				)
+				(hide yes)
+			)
+		)
+		(property "Sim.Pins" "1=A 2=K"
+			(at 217.17 95.25 0)
+			(effects
+				(font
+					(size 1.27 1.27)
+				)
+				(hide yes)
+			)
+		)
 		(pin "1"
 		)
@@
 		)
 		(property "Description" ""
+			(at 179.07 95.25 0)
+			(effects
+				(font
+					(size 1.27 1.27)
+				)
+				(hide yes)
+			)
+		)
+		(property "Sim.Device" "D"
+			(at 179.07 95.25 0)
+			(effects
+				(font
+					(size 1.27 1.27)
+				)
+				(hide yes)
+			)
+		)
+		(property "Sim.Pins" "1=A 2=K"
 			(at 179.07 95.25 0)
 			(effects
@@
 			)
 		)
-		(property "Description" ""
+		(property "Description" "Power symbol creates a global label with name \"+12V\""
 			(at 179.07 76.2 0)
 			(effects
@@
 	(symbol
 		(lib_id "Connector:Conn_01x02_Pin")
-		(at 124.46 105.41 0)
+		(at 154.94 105.41 0)
 		(mirror x)
 		(unit 1)
-		(exclude_from_sim no)
+		(exclude_from_sim yes)
 		(in_bom yes)
 		(on_board yes)
 		(dnp no)
 		(property "Reference" "J1"
-			(at 125.095 110.49 0)
+			(at 155.575 110.49 0)
 			(effects
 				(font
@@
 		)
 		(property "Value" "Conn_01x02_Pin"
-			(at 125.095 107.95 0)
+			(at 155.575 107.95 0)
 			(effects
 				(font
@@
 		)
 		(property "Footprint" "Connector_PinHeader_2.54mm:PinHeader_1x02_P2.54mm_Vertical"
-			(at 124.46 105.41 0)
+			(at 154.94 105.41 0)
 			(effects
 				(font
@@
 		)
 		(property "Datasheet" "~"
-			(at 124.46 105.41 0)
+			(at 154.94 105.41 0)
 			(effects
 				(font
@@
 		)
 		(property "Description" ""
-			(at 124.46 105.41 0)
+			(at 154.94 105.41 0)
 			(effects
 				(font
@@
 			)
 		)
-		(property "Description" ""
+		(property "Description" "Power symbol creates a global label with name \"GND\" , ground"
 			(at 179.07 128.27 0)
 			(effects
@@
 	(symbol
 		(lib_id "PCM_SL_Pin_Headers:PINHD_1x1_Male")
-		(at 252.73 124.46 0)
+		(at 226.06 124.46 0)
 		(unit 1)
-		(exclude_from_sim no)
+		(exclude_from_sim yes)
 		(in_bom yes)
 		(on_board yes)
@@
 		(fields_autoplaced yes)
 		(property "Reference" "J4"
-			(at 255.27 123.1899 0)
+			(at 228.6 123.1899 0)
 			(effects
 				(font
@@
 		)
 		(property "Value" "PINHD_1x1_Male"
-			(at 255.27 125.7299 0)
+			(at 228.6 125.7299 0)
 			(effects
 				(font
@@
 		)
 		(property "Footprint" "Connector_PinHeader_2.54mm:PinHeader_1x01_P2.54mm_Vertical"
-			(at 254 127 0)
+			(at 227.33 127 0)
 			(effects
 				(font
@@
 		)
 		(property "Datasheet" ""
-			(at 252.73 118.11 0)
+			(at 226.06 118.11 0)
 			(effects
 				(font
@@
 		)
 		(property "Description" "Pin Header male with pin space 2.54mm. Pin Count -1"
-			(at 252.73 124.46 0)
+			(at 226.06 124.46 0)
 			(effects
 				(font
@@
 	(symbol
 		(lib_id "power:PWR_FLAG")
-		(at 148.59 81.28 0)
+		(at 166.37 81.28 0)
 		(unit 1)
 		(exclude_from_sim no)
@@
 		(fields_autoplaced yes)
 		(property "Reference" "#FLG01"
-			(at 148.59 79.375 0)
+			(at 166.37 79.375 0)
 			(effects
 				(font
@@
 		)
 		(property "Value" "PWR_FLAG"
-			(at 148.59 77.47 0)
+			(at 166.37 77.47 0)
 			(effects
 				(font
@@
 		)
 		(property "Footprint" ""
-			(at 148.59 81.28 0)
+			(at 166.37 81.28 0)
 			(effects
 				(font
@@
 		)
 		(property "Datasheet" "~"
-			(at 148.59 81.28 0)
-			(effects
-				(font
-					(size 1.27 1.27)
-				)
-				(hide yes)
-			)
-		)
-		(property "Description" ""
-			(at 148.59 81.28 0)
+			(at 166.37 81.28 0)
+			(effects
+				(font
+					(size 1.27 1.27)
+				)
+				(hide yes)
+			)
+		)
+		(property "Description" "Special symbol for telling ERC where power comes from"
+			(at 166.37 81.28 0)
 			(effects
 				(font
@@
 			)
 		)
+		(property "Sim.Device" "NPN"
+			(at 181.61 113.03 0)
+			(effects
+				(font
+					(size 1.27 1.27)
+				)
+				(hide yes)
+			)
+		)
+		(property "Sim.Type" "VBIC"
+			(at 181.61 113.03 0)
+			(effects
+				(font
+					(size 1.27 1.27)
+				)
+				(hide yes)
+			)
+		)
+		(property "Sim.Pins" "1=C 2=B 3=E"
+			(at 181.61 113.03 0)
+			(effects
+				(font
+					(size 1.27 1.27)
+				)
+				(hide yes)
+			)
+		)
 		(pin "1"
 		)
@@
 			(at 214.63 113.03 0)
 			(effects
+				(font
+					(size 1.27 1.27)
+				)
+				(hide yes)
+			)
+		)
+		(property "Sim.Device" "NPN"
+			(at 214.63 113.03 0)
+			(effects
+				(font
+					(size 1.27 1.27)
+				)
+				(hide yes)
+			)
+		)
+		(property "Sim.Type" "VBIC"
+			(at 214.63 113.03 0)
+			(effects
+				(font
+					(size 1.27 1.27)
+				)
+				(hide yes)
+			)
+		)
+		(property "Sim.Pins" "1=C 2=B 3=E"
+			(at 214.63 113.03 0)
+			(effects
